File: Hardware/010_Implementation/CAN_Transceiver.sch (KiCad schematic (older format))
At the start: 15 parts, among them IC1 SN65HVD233-HT, J2 Conn_01x09_Female, Q7 2N7002, U12 FDV304P, U13 FDV304P

Commit message: Changes to Schematic. Button, LEDs and Power Flags
Connections:
- net labels added: +3.3V
- net labels removed: VCC
Changed lines of the file:
@@
 Wire Wire Line
 	9800 3800 10025 3800
-Text GLabel 10025 3100 2    50   Input ~ 0
-GND
-Text GLabel 10025 3800 2    50   Input ~ 0
-VCC
 Wire Wire Line
 	9800 3300 9900 3300
@@
 Text Label 1375 5825 0    50   ~ 0
 EN_CAN
-Text GLabel 2025 6475 3    50   Input ~ 0
-GND
 Wire Wire Line
 	1300 4225 2025 4225
@@
 Connection ~ 2375 4325
 $Comp
-L power:PWR_FLAG #FLG03
+L power:PWR_FLAG #FLG02
 U 1 1 5F5BFD41
 P 1850 3625
-F 0 "#FLG03" H 1850 3700 50  0001 C CNN
+F 0 "#FLG02" H 1850 3700 50  0001 C CNN
 F 1 "PWR_FLAG" H 1850 3798 50  0000 C CNN
 F 2 "" H 1850 3625 50  0001 C CNN
@@
 Text Label 3025 3500 1    50   ~ 0
 EN_CAN
-Text GLabel 6350 4700 3    50   Input ~ 0
-GND
 Text Label 3675 3050 3    50   ~ 0
 CAN_H
@@
 Wire Wire Line
 	3025 2850 3675 2850
+$Comp
+L power:GND #PWR0105
+U 1 1 5F91316D
+P 10025 3100
+F 0 "#PWR0105" H 10025 2850 50  0001 C CNN
+F 1 "GND" H 10030 2927 50  0000 C CNN
+F 2 "" H 10025 3100 50  0001 C CNN
+F 3 "" H 10025 3100 50  0001 C CNN
+	1    10025 3100
+	1    0    0    -1
+$EndComp
+$Comp
+L power:+3.3V #PWR0106
+U 1 1 5F913497
+P 10025 3800
+F 0 "#PWR0106" H 10025 3650 50  0001 C CNN
+F 1 "+3.3V" H 10040 3973 50  0000 C CNN
+F 2 "" H 10025 3800 50  0001 C CNN
+F 3 "" H 10025 3800 50  0001 C CNN
+	1    10025 3800
+	1    0    0    -1
+$EndComp
+$Comp
+L power:GND #PWR0107
+U 1 1 5F9161C7
+P 6350 4700
+F 0 "#PWR0107" H 6350 4450 50  0001 C CNN
+F 1 "GND" H 6355 4527 50  0000 C CNN
+F 2 "" H 6350 4700 50  0001 C CNN
+F 3 "" H 6350 4700 50  0001 C CNN
+	1    6350 4700
+	1    0    0    -1
+$EndComp
+$Comp
+L power:GND #PWR0108
+U 1 1 5F916540
+P 2025 6475
+F 0 "#PWR0108" H 2025 6225 50  0001 C CNN
+F 1 "GND" H 2030 6302 50  0000 C CNN
+F 2 "" H 2025 6475 50  0001 C CNN
+F 3 "" H 2025 6475 50  0001 C CNN
+	1    2025 6475
+	1    0    0    -1
+$EndComp
 $EndSCHEMATC

Commit message: Modified Board Schematic. Optimized supply and switching system through Software
Parts:
- removed J2: Conn_01x09_Female, Connector_Dsub:DSUB-9_Female_Horizontal_P2.77x2.84mm_EdgePinOffset4.94mm_Housed_MountingHolesOffset7.48mm, symbol Connector:Conn_01x09_Female
- removed Q7: 2N7002, Board:SOT23-3, symbol Board:2N7002
- removed R7: 220, Resistor_SMD:R_2512_6332Metric_Pad1.52x3.35mm_HandSolder, symbol Device:R
- removed U12, U13: FDV304P, Board:SOT23-3, symbol Board:FDV304P
- R3: renamed from R8; footprint Resistor_SMD:R_2512_6332Metric_Pad1.52x3.35mm_HandSolder -> Resistor_SMD:R_0805_2012Metric_Pad1.15x1.40mm_HandSolder
- R4: renamed from R9; footprint Resistor_SMD:R_2512_6332Metric_Pad1.52x3.35mm_HandSolder -> Resistor_SMD:R_0805_2012Metric_Pad1.15x1.40mm_HandSolder
Connections:
- net labels added: BUS_H, BUS_L
- net labels removed: CAN_GND, CAN_H, CAN_L, EN_CAN, EN_Transceiver, OBD_GND, OBD_H, OBD_L, OBD_VDD, Signal_H, Signal_L
- wire segments 83 -> 58
- no-connect marks 4 -> 0
Other:
- note removed: "CAN_GND Decoupler"
- note removed: "DSUB-9 Connector\n"
- moved on the sheet: C3, C4, C5, C6, IC1, R3, R4

Commit message: PCB Updated
Parts:
- removed D1, D2: SD05_SOD323, Diode_SMD:D_SOD-323, symbol Diode:SD05_SOD323
- added D1: PESD1CAN, Board:SOT23-3, symbol Board:PESD1CAN
Connections:
- wire segments 58 -> 55
Changed lines of the file:
@@
 	5075 4375 5075 4050
-Wire Wire Line
-	2800 2525 3400 2525
-Wire Wire Line
-	2800 3450 3400 3450
-Connection ~ 3400 3450
 Wire Wire Line
 	3925 4050 4450 4050
@@
 Connection ~ 4450 4050
 Wire Wire Line
-	3400 3025 3400 3100
-Connection ~ 3400 3025
-Wire Wire Line
 	3700 3025 3700 4050
-Wire Wire Line
-	3400 3025 3700 3025
-Wire Wire Line
-	3400 3450 4450 3450
-Wire Wire Line
-	3400 3400 3400 3450
-Wire Wire Line
-	3400 2525 3925 2525
-Connection ~ 3400 2525
-Wire Wire Line
-	3400 2650 3400 2525
-Wire Wire Line
-	3400 2950 3400 3025
 Wire Wire Line
 	3925 2525 4675 2525
@@
 Wire Wire Line
 	4675 3450 4675 3300
-$Comp
-L Diode:SD05_SOD323 D2
-U 1 1 5F5F1395
-P 3400 3250
-F 0 "D2" V 3354 3329 50  0000 L CNN
-F 1 "SD05_SOD323" V 3445 3329 50  0000 L CNN
-F 2 "Diode_SMD:D_SOD-323" H 3400 3050 50  0001 C CNN
-F 3 "https://www.littelfuse.com/~/media/electronics/datasheets/tvs_diode_arrays/littelfuse_tvs_diode_array_sd_c_datasheet.pdf.pdf" H 3400 3250 50  0001 C CNN
-	1    3400 3250
-	0    1    1    0
-$EndComp
-$Comp
-L Diode:SD05_SOD323 D1
-U 1 1 5F5F138F
-P 3400 2800
-F 0 "D1" V 3446 2721 50  0000 R CNN
-F 1 "SD05_SOD323" V 3355 2721 50  0000 R CNN
-F 2 "Diode_SMD:D_SOD-323" H 3400 2600 50  0001 C CNN
-F 3 "https://www.littelfuse.com/~/media/electronics/datasheets/tvs_diode_arrays/littelfuse_tvs_diode_array_sd_c_datasheet.pdf.pdf" H 3400 2800 50  0001 C CNN
-	1    3400 2800
-	0    -1   -1   0
-$EndComp
 Wire Wire Line
 	4450 3800 4450 4050
@@
 Text HLabel 2800 3450 0    50   BiDi ~ 0
 BUS_L
+$Comp
+L Board:PESD1CAN D1
+U 1 1 5FA9220A
+P 3100 3225
+F 0 "D1" H 3300 3792 50  0000 C CNN
+F 1 "PESD1CAN" H 3300 3701 50  0000 C CNN
+F 2 "Board:SOT23-3" H 3100 3225 50  0001 L BNN
+F 3 "" H 3100 3225 50  0001 L BNN
+F 4 "DIO-12501" H 3100 3225 50  0001 L BNN "PROD_ID"
+	1    3100 3225
+	1    0    0    -1
+$EndComp
+Wire Wire Line
+	2800 2525 2900 2525
+Wire Wire Line
+	2800 3450 2900 3450
+Wire Wire Line
+	2900 3125 2900 3450
+Connection ~ 2900 3450
+Wire Wire Line
+	2900 3450 4450 3450
+Wire Wire Line
+	2900 2925 2900 2525
+Connection ~ 2900 2525
+Wire Wire Line
+	2900 2525 3925 2525
 $EndSCHEMATC

Commit message: Board version 4
Parts:
- removed L1: L_Core_Ferrite_Coupled, Transformer_THT:Transformer_Toroid_Horizontal_D9.0mm_Amidon-T30, symbol Device:L_Core_Ferrite_Coupled
- added L2: 744242220, SamacSys_Parts:WE-SLM77, symbol SamacSys_Parts:744242220
- added R4, R5: 0, Resistor_SMD:R_0603_1608Metric_Pad1.05x0.95mm_HandSolder, symbol Device:R
- C4: renamed from C3; footprint Capacitor_SMD:C_1812_4532Metric_Pad1.30x3.40mm_HandSolder -> Capacitor_SMD:C_0603_1608Metric_Pad1.05x0.95mm_HandSolder
- C5: renamed from C4; footprint Capacitor_SMD:C_1812_4532Metric_Pad1.30x3.40mm_HandSolder -> Capacitor_SMD:C_0603_1608Metric_Pad1.05x0.95mm_HandSolder
- C6: renamed from C5; footprint Capacitor_SMD:C_1812_4532Metric_Pad1.30x3.40mm_HandSolder -> Capacitor_SMD:C_0603_1608Metric_Pad1.05x0.95mm_HandSolder
- C7: renamed from C6; footprint Capacitor_SMD:C_1812_4532Metric_Pad1.30x3.40mm_HandSolder -> Capacitor_SMD:C_0603_1608Metric_Pad1.05x0.95mm_HandSolder
- renumbered R3 to R6, R4 to R7
Connections:
- wire segments 55 -> 62
Other:
- moved on the sheet: C4, C5
Changed lines of the file:
@@
 	8525 3075 8625 3075
 $Comp
-L power:GND #PWR03
+L power:GND #PWR06
 U 1 1 5F9161C7
 P 5075 4375
-F 0 "#PWR03" H 5075 4125 50  0001 C CNN
+F 0 "#PWR06" H 5075 4125 50  0001 C CNN
 F 1 "GND" H 5080 4202 50  0000 C CNN
 F 2 "" H 5075 4375 50  0001 C CNN
@@
 $EndComp
 $Comp
-L power:+3.3V #PWR05
+L power:+3.3V #PWR08
 U 1 1 5F913497
 P 8750 3600
-F 0 "#PWR05" H 8750 3450 50  0001 C CNN
+F 0 "#PWR08" H 8750 3450 50  0001 C CNN
 F 1 "+3.3V" H 8765 3773 50  0000 C CNN
 F 2 "" H 8750 3600 50  0001 C CNN
@@
 $EndComp
 $Comp
-L power:GND #PWR04
+L power:GND #PWR07
 U 1 1 5F91316D
 P 8750 2775
-F 0 "#PWR04" H 8750 2525 50  0001 C CNN
+F 0 "#PWR07" H 8750 2525 50  0001 C CNN
 F 1 "GND" H 8755 2602 50  0000 C CNN
 F 2 "" H 8750 2775 50  0001 C CNN
@@
 Connection ~ 3925 2525
 Wire Wire Line
-	3925 2525 3925 3500
-Wire Wire Line
-	4675 3100 4875 3100
-Wire Wire Line
-	4675 2525 4675 3100
+	3925 2525 3925 3600
 Wire Wire Line
 	4450 3450 4675 3450
 Connection ~ 4450 3450
 Wire Wire Line
-	4450 3500 4450 3450
-Wire Wire Line
-	4675 3300 4875 3300
-Wire Wire Line
-	4675 3450 4675 3300
-Wire Wire Line
-	4450 3800 4450 4050
+	4450 3600 4450 3450
+Wire Wire Line
+	4450 3900 4450 4050
 Connection ~ 3925 4050
 Wire Wire Line
 	3925 4050 3700 4050
 Wire Wire Line
-	3925 3800 3925 4050
-$Comp
-L Device:C C3
+	3925 3900 3925 4050
+$Comp
+L Device:C C4
 U 1 1 5F5F1385
-P 3925 3650
-F 0 "C3" H 4040 3696 50  0000 L CNN
-F 1 "100p" H 4040 3605 50  0000 L CNN
-F 2 "Capacitor_SMD:C_1812_4532Metric_Pad1.30x3.40mm_HandSolder" H 3963 3500 50  0001 C CNN
-F 3 "~" H 3925 3650 50  0001 C CNN
-	1    3925 3650
-	1    0    0    -1
-$EndComp
-$Comp
-L Device:C C4
+P 3925 3750
+F 0 "C4" H 4040 3796 50  0000 L CNN
+F 1 "100p" H 4040 3705 50  0000 L CNN
+F 2 "Capacitor_SMD:C_0603_1608Metric_Pad1.05x0.95mm_HandSolder" H 3963 3600 50  0001 C CNN
+F 3 "~" H 3925 3750 50  0001 C CNN
+	1    3925 3750
+	1    0    0    -1
+$EndComp
+$Comp
+L Device:C C5
 U 1 1 5F5F137F
-P 4450 3650
-F 0 "C4" H 4565 3696 50  0000 L CNN
-F 1 "100p" H 4565 3605 50  0000 L CNN
-F 2 "Capacitor_SMD:C_1812_4532Metric_Pad1.30x3.40mm_HandSolder" H 4488 3500 50  0001 C CNN
-F 3 "~" H 4450 3650 50  0001 C CNN
-	1    4450 3650
+P 4450 3750
+F 0 "C5" H 4565 3796 50  0000 L CNN
+F 1 "100p" H 4565 3705 50  0000 L CNN
+F 2 "Capacitor_SMD:C_0603_1608Metric_Pad1.05x0.95mm_HandSolder" H 4488 3600 50  0001 C CNN
+F 3 "~" H 4450 3750 50  0001 C CNN
+	1    4450 3750
 	1    0    0    -1
 $EndComp
@@
 Wire Wire Line
 	5525 3800 5750 3800
-Wire Wire Line
-	5525 3300 5525 3800
-Wire Wire Line
-	5275 3300 5525 3300
 Connection ~ 5750 2650
 Wire Wire Line
 	5525 2650 5750 2650
-Wire Wire Line
-	5525 3100 5525 2650
-Wire Wire Line
-	5275 3100 5525 3100
-$Comp
-L Device:L_Core_Ferrite_Coupled L1
-U 1 1 5F5F1371
-P 5075 3200
-F 0 "L1" H 5075 2875 50  0000 C CNN
-F 1 "L_Core_Ferrite_Coupled" H 5075 2966 50  0000 C CNN
-F 2 "Transformer_THT:Transformer_Toroid_Horizontal_D9.0mm_Amidon-T30" H 5075 3200 50  0001 C CNN
-F 3 "~" H 5075 3200 50  0001 C CNN
-	1    5075 3200
-	-1   0    0    -1
-$EndComp
 Connection ~ 6200 3800
 Wire Wire Line
@@
 	5750 3050 5750 2650
 $Comp
-L Device:C C5
+L Device:C C6
 U 1 1 5F5F1365
 P 5750 3200
-F 0 "C5" H 5865 3246 50  0000 L CNN
+F 0 "C6" H 5865 3246 50  0000 L CNN
 F 1 "100p" H 5865 3155 50  0000 L CNN
-F 2 "Capacitor_SMD:C_1812_4532Metric_Pad1.30x3.40mm_HandSolder" H 5788 3050 50  0001 C CNN
+F 2 "Capacitor_SMD:C_0603_1608Metric_Pad1.05x0.95mm_HandSolder" H 5788 3050 50  0001 C CNN
 F 3 "~" H 5750 3200 50  0001 C CNN
 	1    5750 3200
@@
 	6200 3675 6200 3800
 $Comp
-L Device:C C6
+L Device:C C7
 U 1 1 5F5F1351
 P 6700 3800
-F 0 "C6" H 6815 3846 50  0000 L CNN
+F 0 "C7" H 6815 3846 50  0000 L CNN
 F 1 "4n7" H 6815 3755 50  0000 L CNN
-F 2 "Capacitor_SMD:C_1812_4532Metric_Pad1.30x3.40mm_HandSolder" H 6738 3650 50  0001 C CNN
+F 2 "Capacitor_SMD:C_0603_1608Metric_Pad1.05x0.95mm_HandSolder" H 6738 3650 50  0001 C CNN
 F 3 "~" H 6700 3800 50  0001 C CNN
 	1    6700 3800
@@
 $EndComp
 $Comp
-L Device:R R4
+L Device:R R7
 U 1 1 5F5F134B
 P 6200 3525
-F 0 "R4" H 6270 3571 50  0000 L CNN
+F 0 "R7" H 6270 3571 50  0000 L CNN
 F 1 "62" H 6270 3480 50  0000 L CNN
 F 2 "Resistor_SMD:R_0805_2012Metric_Pad1.15x1.40mm_HandSolder" V 6130 3525 50  0001 C CNN
@@
 $EndComp
 $Comp
-L Device:R R3
+L Device:R R6
 U 1 1 5F5F1345
 P 6200 2900
-F 0 "R3" H 6270 2946 50  0000 L CNN
+F 0 "R6" H 6270 2946 50  0000 L CNN
 F 1 "62" H 6270 2855 50  0000 L CNN
 F 2 "Resistor_SMD:R_0805_2012Metric_Pad1.15x1.40mm_HandSolder" V 6130 2900 50  0001 C CNN
@@
 Wire Wire Line
 	2900 2525 3925 2525
+$Comp
+L SamacSys_Parts:744242220 L2
+U 1 1 5FA954C1
+P 5500 3150
+F 0 "L2" H 5900 3415 50  0000 C CNN
+F 1 "744242220" H 5900 3324 50  0000 C CNN
+F 2 "SamacSys_Parts:WE-SLM77" H 6150 3250 50  0001 L CNN
+F 3 "https://componentsearchengine.com/Datasheets/1/744242220.pdf" H 6150 3150 50  0001 L CNN
+F 4 "Wurth WE-SLM Series Wire-wound SMD Inductor with a Ferrite Core, 22 uH +50/-30 300mA Idc" H 6150 3050 50  0001 L CNN "Description"
+F 5 "" H 6150 2950 50  0001 L CNN "Height"
+F 6 "710-744242220" H 6150 2850 50  0001 L CNN "Mouser Part Number"
+F 7 "https://www.mouser.com/Search/Refine.aspx?Keyword=710-744242220" H 6150 2750 50  0001 L CNN "Mouser Price/Stock"
+F 8 "Wurth Elektronik" H 6150 2650 50  0001 L CNN "Manufacturer_Name"
+F 9 "744242220" H 6150 2550 50  0001 L CNN "Manufacturer_Part_Number"
+	1    5500 3150
+	-1   0    0    -1
+$EndComp
+Wire Wire Line
+	5500 3150 5525 3150
+Wire Wire Line
+	5500 3250 5525 3250
+Wire Wire Line
+	5525 3250 5525 3550
+Wire Wire Line
+	4700 3250 4675 3250
+Wire Wire Line
+	4675 3250 4675 3450
+Wire Wire Line
+	4700 3150 4675 3150
+Wire Wire Line
+	4675 2525 4675 2650
+$Comp
+L Device:R R4
+U 1 1 5FB22CE5
+P 5100 2650
+F 0 "R4" V 4893 2650 50  0000 C CNN
+F 1 "0" V 4984 2650 50  0000 C CNN
+F 2 "Resistor_SMD:R_0603_1608Metric_Pad1.05x0.95mm_HandSolder" V 5030 2650 50  0001 C CNN
+F 3 "~" H 5100 2650 50  0001 C CNN
+	1    5100 2650
+	0    1    1    0
+$EndComp
+$Comp
+L Device:R R5
+U 1 1 5FB23167
+P 5100 3550
+F 0 "R5" V 4893 3550 50  0000 C CNN
+F 1 "0" V 4984 3550 50  0000 C CNN
+F 2 "Resistor_SMD:R_0603_1608Metric_Pad1.05x0.95mm_HandSolder" V 5030 3550 50  0001 C CNN
+F 3 "~" H 5100 3550 50  0001 C CNN
+	1    5100 3550
+	0    1    1    0
+$EndComp
+Wire Wire Line
+	4950 2650 4675 2650
+Wire Wire Line
+	5250 2650 5525 2650
+Wire Wire Line
+	5250 3550 5525 3550
+Connection ~ 5525 3550
+Wire Wire Line
+	5525 3550 5525 3800
+Wire Wire Line
+	4950 3550 4675 3550
+Wire Wire Line
+	4675 3550 4675 3450
+Connection ~ 4675 3450
+Connection ~ 4675 2650
+Connection ~ 5525 2650
+Wire Wire Line
+	5525 2650 5525 3150
+Wire Wire Line
+	4675 2650 4675 3150
 $EndSCHEMATC

Commit message: Board version 4.1
Parts:
- L2: symbol SamacSys_Parts:744242220 -> Board-rescue:744242220-SamacSys_Parts
Connections:
- wire segments 62 -> 65
Changed lines of the file:
@@
 Wire Wire Line
 	8525 3475 8525 3600
-Connection ~ 8625 2975
-Wire Wire Line
-	8625 3075 8625 2975
-Wire Wire Line
-	8525 3075 8625 3075
 $Comp
 L power:GND #PWR06
@@
 L power:GND #PWR07
 U 1 1 5F91316D
-P 8750 2775
-F 0 "#PWR07" H 8750 2525 50  0001 C CNN
-F 1 "GND" H 8755 2602 50  0000 C CNN
-F 2 "" H 8750 2775 50  0001 C CNN
-F 3 "" H 8750 2775 50  0001 C CNN
-	1    8750 2775
+P 8900 2950
+F 0 "#PWR07" H 8900 2700 50  0001 C CNN
+F 1 "GND" H 8905 2777 50  0000 C CNN
+F 2 "" H 8900 2950 50  0001 C CNN
+F 3 "" H 8900 2950 50  0001 C CNN
+	1    8900 2950
 	1    0    0    -1
 $EndComp
@@
 Transceiver
 Wire Wire Line
-	8625 2775 8750 2775
-Connection ~ 8625 2775
-Wire Wire Line
-	8625 2975 8625 2775
-Wire Wire Line
-	8525 2975 8625 2975
-Wire Wire Line
 	8525 3600 8750 3600
-Wire Wire Line
-	8525 2775 8625 2775
 Wire Wire Line
 	8525 3275 9175 3275
@@
 	2900 2525 3925 2525
 $Comp
-L SamacSys_Parts:744242220 L2
+L Board-rescue:744242220-SamacSys_Parts L2
 U 1 1 5FA954C1
 P 5500 3150
+AR Path="/5FA954C1" Ref="L2"  Part="1"
+AR Path="/5F562A6B/5FA954C1" Ref="L2"  Part="1"
 F 0 "L2" H 5900 3415 50  0000 C CNN
 F 1 "744242220" H 5900 3324 50  0000 C CNN
@@
 Wire Wire Line
 	4675 2650 4675 3150
+$Comp
+L power:GND #PWR0101
+U 1 1 5FAB0F55
+P 8900 2800
+F 0 "#PWR0101" H 8900 2550 50  0001 C CNN
+F 1 "GND" H 8905 2627 50  0000 C CNN
+F 2 "" H 8900 2800 50  0001 C CNN
+F 3 "" H 8900 2800 50  0001 C CNN
+	1    8900 2800
+	1    0    0    -1
+$EndComp
+$Comp
+L power:GND #PWR0102
+U 1 1 5FAB15C4
+P 8900 2650
+F 0 "#PWR0102" H 8900 2400 50  0001 C CNN
+F 1 "GND" H 8905 2477 50  0000 C CNN
+F 2 "" H 8900 2650 50  0001 C CNN
+F 3 "" H 8900 2650 50  0001 C CNN
+	1    8900 2650
+	1    0    0    -1
+$EndComp
+Wire Wire Line
+	8815 3075 8815 2950
+Wire Wire Line
+	8815 2950 8900 2950
+Wire Wire Line
+	8525 3075 8815 3075
+Wire Wire Line
+	8525 2975 8775 2975
+Wire Wire Line
+	8775 2975 8775 2800
+Wire Wire Line
+	8775 2800 8900 2800
+Wire Wire Line
+	8525 2775 8740 2775
+Wire Wire Line
+	8740 2775 8740 2650
+Wire Wire Line
+	8740 2650 8900 2650
 $EndSCHEMATC

Commit message: Board Version 4.2
Parts:
- added R21: 0, symbol Device:R
- R4, R5: NP (none) -> NP
Connections:
- net BUS_L: now also C5.2; no longer C5.1
- net GND: now also C5.1, R21.2; no longer C5.2, IC1.8 (RS)
- new net: IC1.8 (RS), R21.1
Other:
- moved on the sheet: C4, C5, C6, C7, D1, IC1, L2, R4, R5, R6, R7

Commit message: Board Version 5
Parts:
- C4, C5, C6: footprint Capacitor_SMD:C_0603_1608Metric_Pad1.05x0.95mm_HandSolder -> Capacitor_SMD:C_0603_1608Metric_Pad1.08x0.95mm_HandSolder
- C7: value 4n7 -> 4n; footprint Capacitor_SMD:C_0603_1608Metric_Pad1.05x0.95mm_HandSolder -> Capacitor_SMD:C_0603_1608Metric_Pad1.08x0.95mm_HandSolder
- D1: Vorhanden (none) -> Yes
- R21: footprint (none) -> Resistor_SMD:R_0603_1608Metric_Pad0.98x0.95mm_HandSolder
- R4, R5: footprint Resistor_SMD:R_0603_1608Metric_Pad1.05x0.95mm_HandSolder -> Resistor_SMD:R_0603_1608Metric_Pad0.98x0.95mm_HandSolder
- R6, R7: footprint Resistor_SMD:R_0805_2012Metric_Pad1.15x1.40mm_HandSolder -> Resistor_SMD:R_0603_1608Metric_Pad0.98x0.95mm_HandSolder
Changed lines of the file:
@@
 F 0 "C4" H 3300 3796 50  0000 L CNN
 F 1 "100p" H 3300 3705 50  0000 L CNN
-F 2 "Capacitor_SMD:C_0603_1608Metric_Pad1.05x0.95mm_HandSolder" H 3223 3600 50  0001 C CNN
+F 2 "Capacitor_SMD:C_0603_1608Metric_Pad1.08x0.95mm_HandSolder" H 3223 3600 50  0001 C CNN
 F 3 "~" H 3185 3750 50  0001 C CNN
 	1    3185 3750
@@
 F 0 "C5" H 3300 3251 50  0000 L CNN
 F 1 "100p" H 3300 3160 50  0000 L CNN
-F 2 "Capacitor_SMD:C_0603_1608Metric_Pad1.05x0.95mm_HandSolder" H 3223 3055 50  0001 C CNN
+F 2 "Capacitor_SMD:C_0603_1608Metric_Pad1.08x0.95mm_HandSolder" H 3223 3055 50  0001 C CNN
 F 3 "~" H 3185 3205 50  0001 C CNN
 	1    3185 3205
@@
 F 0 "C6" H 5450 3526 50  0000 L CNN
 F 1 "100p" H 5450 3435 50  0000 L CNN
-F 2 "Capacitor_SMD:C_0603_1608Metric_Pad1.05x0.95mm_HandSolder" H 5373 3330 50  0001 C CNN
+F 2 "Capacitor_SMD:C_0603_1608Metric_Pad1.08x0.95mm_HandSolder" H 5373 3330 50  0001 C CNN
 F 3 "~" H 5335 3480 50  0001 C CNN
 	1    5335 3480
@@
 P 6240 3455
 F 0 "C7" H 6355 3501 50  0000 L CNN
-F 1 "4n7" H 6355 3410 50  0000 L CNN
-F 2 "Capacitor_SMD:C_0603_1608Metric_Pad1.05x0.95mm_HandSolder" H 6278 3305 50  0001 C CNN
+F 1 "4n" H 6355 3410 50  0000 L CNN
+F 2 "Capacitor_SMD:C_0603_1608Metric_Pad1.08x0.95mm_HandSolder" H 6278 3305 50  0001 C CNN
 F 3 "~" H 6240 3455 50  0001 C CNN
 	1    6240 3455
@@
 F 0 "R7" H 6005 3206 50  0000 L CNN
 F 1 "62" H 6005 3115 50  0000 L CNN
-F 2 "Resistor_SMD:R_0805_2012Metric_Pad1.15x1.40mm_HandSolder" V 5865 3160 50  0001 C CNN
+F 2 "Resistor_SMD:R_0603_1608Metric_Pad0.98x0.95mm_HandSolder" V 5865 3160 50  0001 C CNN
 F 3 "~" H 5935 3160 50  0001 C CNN
 	1    5935 3160
@@
 F 0 "R6" H 6005 3801 50  0000 L CNN
 F 1 "62" H 6005 3710 50  0000 L CNN
-F 2 "Resistor_SMD:R_0805_2012Metric_Pad1.15x1.40mm_HandSolder" V 5865 3755 50  0001 C CNN
+F 2 "Resistor_SMD:R_0603_1608Metric_Pad0.98x0.95mm_HandSolder" V 5865 3755 50  0001 C CNN
 F 3 "~" H 5935 3755 50  0001 C CNN
 	1    5935 3755
@@
 F 1 "PESD1CAN" H 2445 3205 50  0000 C CNN
 F 2 "Board:SOT23-3" H 2240 3255 50  0001 L BNN
-F 3 "" H 2240 3255 50  0001 L BNN
+F 3 "https://assets.nexperia.com/documents/data-sheet/PESD1CAN.pdf" H 2240 3255 50  0001 L BNN
 F 4 "DIO-12501" H 2240 3255 50  0001 L BNN "PROD_ID"
+F 5 "Yes" H 2240 3255 50  0001 C CNN "Vorhanden"
 	1    2240 3255
 	1    0    0    1
@@
 F 0 "R4" V 4660 4200 50  0000 C CNN
 F 1 "0" V 4444 4205 50  0000 C CNN
-F 2 "Resistor_SMD:R_0603_1608Metric_Pad1.05x0.95mm_HandSolder" V 4490 4205 50  0001 C CNN
+F 2 "Resistor_SMD:R_0603_1608Metric_Pad0.98x0.95mm_HandSolder" V 4490 4205 50  0001 C CNN
 F 3 "~" H 4560 4205 50  0001 C CNN
 F 4 "NP" V 4560 4205 50  0000 C CNN "NP"
@@
 F 0 "R5" V 4660 2700 50  0000 C CNN
 F 1 "0" V 4444 2705 50  0000 C CNN
-F 2 "Resistor_SMD:R_0603_1608Metric_Pad1.05x0.95mm_HandSolder" V 4490 2705 50  0001 C CNN
+F 2 "Resistor_SMD:R_0603_1608Metric_Pad0.98x0.95mm_HandSolder" V 4490 2705 50  0001 C CNN
 F 3 "~" H 4560 2705 50  0001 C CNN
 F 4 "NP" V 4560 2705 50  0000 C CNN "NP"
@@
 F 1 "SN65HVD233-HT" H 7805 4035 50  0000 C CNN
 F 2 "Board:SOIC127P600X175" H 7805 3485 50  0001 L BNN
-F 3 "" H 7805 3485 50  0001 C CNN
+F 3 "https://www.ti.com/lit/ds/symlink/sn65hvd233-ht.pdf?HQS=TI-null-null-alldatasheets-df-pf-SEP-wwe" H 7805 3485 50  0001 C CNN
 	1    7805 3485
 	-1   0    0    -1
@@
 F 0 "R21" H 8825 4021 50  0000 L CNN
 F 1 "0" H 8825 3930 50  0000 L CNN
-F 2 "" V 8685 3975 50  0001 C CNN
+F 2 "Resistor_SMD:R_0603_1608Metric_Pad0.98x0.95mm_HandSolder" V 8685 3975 50  0001 C CNN
 F 3 "~" H 8755 3975 50  0001 C CNN
 	1    8755 3975

Commit message: Board Version 6
Parts:
- added C17: 100n, Capacitor_SMD:C_0603_1608Metric_Pad1.05x0.95mm_HandSolder, symbol Device:C
Connections:
- net +3V3: now also C17.1
- net GND: now also C17.2
Changed lines of the file:
@@
 L power:+3.3V #PWR08
 U 1 1 5F913497
-P 8850 3150
-F 0 "#PWR08" H 8850 3000 50  0001 C CNN
-F 1 "+3.3V" H 8865 3323 50  0000 C CNN
-F 2 "" H 8850 3150 50  0001 C CNN
-F 3 "" H 8850 3150 50  0001 C CNN
-	1    8850 3150
+P 9450 2050
+F 0 "#PWR08" H 9450 1900 50  0001 C CNN
+F 1 "+3.3V" H 9465 2223 50  0000 C CNN
+F 2 "" H 9450 2050 50  0001 C CNN
+F 3 "" H 9450 2050 50  0001 C CNN
+	1    9450 2050
 	-1   0    0    -1
 $EndComp
@@
 $EndComp
 Wire Wire Line
-	8505 3185 8850 3185
-Wire Wire Line
-	8850 3185 8850 3150
-Wire Wire Line
 	8520 3885 8520 4300
 $Comp
@@
 Wire Wire Line
 	6390 3455 6600 3455
+$Comp
+L Device:C C17
+U 1 1 5FBA0AB2
+P 9450 2425
+F 0 "C17" H 9565 2471 50  0000 L CNN
+F 1 "100n" H 9565 2380 50  0000 L CNN
+F 2 "Capacitor_SMD:C_0603_1608Metric_Pad1.05x0.95mm_HandSolder" H 9488 2275 50  0001 C CNN
+F 3 "~" H 9450 2425 50  0001 C CNN
+	1    9450 2425
+	1    0    0    -1
+$EndComp
+Wire Wire Line
+	9450 2050 9450 2175
+Wire Wire Line
+	9450 2175 8900 2175
+Connection ~ 9450 2175
+Wire Wire Line
+	9450 2175 9450 2275
+Wire Wire Line
+	8505 3185 8900 3185
+Wire Wire Line
+	8900 2175 8900 3185
+Wire Wire Line
+	9450 2575 9450 2700
+$Comp
+L power:GND #PWR0104
+U 1 1 5FBA5D45
+P 9450 2700
+F 0 "#PWR0104" H 9450 2450 50  0001 C CNN
+F 1 "GND" H 9455 2527 50  0000 C CNN
+F 2 "" H 9450 2700 50  0001 C CNN
+F 3 "" H 9450 2700 50  0001 C CNN
+	1    9450 2700
+	1    0    0    -1
+$EndComp
 $EndSCHEMATC
