File: Hardware/010_Implementation/CAN_Transceiver.sch (KiCad schematic (older format))
At the start: 13 parts, among them IC1 SN65HVD233-HT

Commit message: Moved Pi-Filter to the top section. Added alignment marks on the back layer.
Parts:
- C17: footprint Capacitor_SMD:C_0603_1608Metric_Pad1.05x0.95mm_HandSolder -> Capacitor_SMD:C_0603_1608Metric_Pad1.08x0.95mm_HandSolder
Changed lines of the file:
@@
 F 0 "C17" H 9565 2471 50  0000 L CNN
 F 1 "100n" H 9565 2380 50  0000 L CNN
-F 2 "Capacitor_SMD:C_0603_1608Metric_Pad1.05x0.95mm_HandSolder" H 9488 2275 50  0001 C CNN
+F 2 "Capacitor_SMD:C_0603_1608Metric_Pad1.08x0.95mm_HandSolder" H 9488 2275 50  0001 C CNN
 F 3 "~" H 9450 2425 50  0001 C CNN
 	1    9450 2425
