File: Hardware/010_Implementation/Board.kicad_pcb (KiCad board)
At the start: 2 copper layers, 123.2 x 44.5 mm, 45 parts, among them IC1 SN65HVD233-HT, J1 2606-3356, J2 Conn_02x05_Odd_Even, J3 Conn_01x09_Female, K1 G5V-2-DC5, K2 G5V-2-DC5, Q1 BC817, SW1 SW_Push, U1 TPS62163DGK, U2 ESP32-DEVKITC-32D

Commit message: Board Version 5
Parts:
- added C10: 100n, Capacitor_SMD:C_0603_1608Metric_Pad1.08x0.95mm_HandSolder, F.Cu at (161.2, 104.7)
- added C11: 100n, Capacitor_SMD:C_0603_1608Metric_Pad1.08x0.95mm_HandSolder, F.Cu at (82.1, 113.8)
- added C12: 1u, Capacitor_SMD:C_0603_1608Metric_Pad1.08x0.95mm_HandSolder, F.Cu at (170.3, 98.3)
- added C13: 100n, Capacitor_SMD:C_0603_1608Metric_Pad1.08x0.95mm_HandSolder, F.Cu at (167.1, 98.3)
- added C14: 100n, Capacitor_SMD:C_0603_1608Metric_Pad1.08x0.95mm_HandSolder, F.Cu at (170.3, 102.6)
- added C15: 1u, Capacitor_SMD:C_0603_1608Metric_Pad1.08x0.95mm_HandSolder, F.Cu at (167.1, 103.0)
- added C16: 10u, Capacitor_SMD:C_1206_3216Metric_Pad1.33x1.80mm_HandSolder, F.Cu at (132.2, 104.1)
- added C9: 100n, Capacitor_SMD:C_0603_1608Metric_Pad1.08x0.95mm_HandSolder, F.Cu at (134.5, 104.2)
- added D8: SMAJ16A, Diode_SMD:D_SMA, F.Cu at (128.9, 104.0)
- added F1: R452002, Fuse:Fuse_2512_6332Metric_Pad1.52x3.35mm_HandSolder, F.Cu at (122.5, 103.8)
- added FB1: Ferrite_Bead, Inductor_SMD:L_0603_1608Metric_Pad1.05x0.95mm_HandSolder, F.Cu at (134.6, 100.6)
- added FB2: Ferrite_Bead, Inductor_SMD:L_0603_1608Metric_Pad1.05x0.95mm_HandSolder, F.Cu at (160.3, 102.1)
- added R19: 953k, Resistor_SMD:R_0603_1608Metric_Pad0.98x0.95mm_HandSolder, F.Cu at (154.1, 101.5)
- added R20: 180k, Resistor_SMD:R_0603_1608Metric_Pad0.98x0.95mm_HandSolder, F.Cu at (154.1, 105.0)
- added R21: 0, Resistor_SMD:R_0603_1608Metric_Pad0.98x0.95mm_HandSolder, F.Cu at (75.0, 84.1)
- C1: value 10n -> 100n; footprint Capacitor_SMD:C_0603_1608Metric_Pad1.05x0.95mm_HandSolder -> Capacitor_SMD:C_0603_1608Metric_Pad1.08x0.95mm_HandSolder; moved to B.Cu
- C2, C3: footprint Capacitor_SMD:C_0603_1608Metric_Pad1.05x0.95mm_HandSolder -> Capacitor_SMD:C_1206_3216Metric_Pad1.33x1.80mm_HandSolder
- C4, C5, C6: footprint Capacitor_SMD:C_0603_1608Metric_Pad1.05x0.95mm_HandSolder -> Capacitor_SMD:C_0603_1608Metric_Pad1.08x0.95mm_HandSolder; moved to F.Cu
- C7: value 4n7 -> 4n; footprint Capacitor_SMD:C_0603_1608Metric_Pad1.05x0.95mm_HandSolder -> Capacitor_SMD:C_0603_1608Metric_Pad1.08x0.95mm_HandSolder; moved to F.Cu
- C8: footprint Capacitor_SMD:C_0603_1608Metric_Pad1.05x0.95mm_HandSolder -> Capacitor_SMD:C_0603_1608Metric_Pad1.08x0.95mm_HandSolder
- D1, J1, L2: moved to F.Cu
- J2: value Conn_02x05_Odd_Even -> JTAG Jumper Pins
- J3: value Conn_01x09_Female -> DSUB9
- Q1: moved to B.Cu
- R1, R17, R18, R2: footprint Resistor_SMD:R_0805_2012Metric_Pad1.15x1.40mm_HandSolder -> Resistor_SMD:R_0603_1608Metric_Pad0.98x0.95mm_HandSolder; moved to B.Cu
- R10, R11, R12, R13, R14, R15, R16, R9: footprint Resistor_SMD:R_0805_2012Metric_Pad1.15x1.40mm_HandSolder -> Resistor_SMD:R_0603_1608Metric_Pad0.98x0.95mm_HandSolder
- R3: value 100k -> 10k; footprint Resistor_SMD:R_0805_2012Metric_Pad1.15x1.40mm_HandSolder -> Resistor_SMD:R_0603_1608Metric_Pad0.98x0.95mm_HandSolder
- R4, R5: footprint Resistor_SMD:R_0603_1608Metric_Pad1.05x0.95mm_HandSolder -> Resistor_SMD:R_0603_1608Metric_Pad0.98x0.95mm_HandSolder; moved to F.Cu
- R6, R7: footprint Resistor_SMD:R_0805_2012Metric_Pad1.15x1.40mm_HandSolder -> Resistor_SMD:R_0603_1608Metric_Pad0.98x0.95mm_HandSolder; moved to F.Cu
- R8: value 2.2k -> 1k; footprint Resistor_SMD:R_0805_2012Metric_Pad1.15x1.40mm_HandSolder -> Resistor_SMD:R_0603_1608Metric_Pad0.98x0.95mm_HandSolder
- U1: value TPS62163DGK -> TPS62170DGK
- moved U2 108.7 mm to (101.1, 93.4), turned to 180 degrees
- moved J1 108.2 mm to (123.6, 79.0), turned to 0 degrees
- moved R5 98.4 mm to (64.4, 75.8)
- moved C6 95.3 mm to (69.8, 80.3), turned to 90 degrees
- moved C7 95.1 mm to (74.2, 80.3)
- moved L2 94.8 mm to (64.3, 80.3)
- moved R7 94.4 mm to (72.0, 78.5)
- moved IC1 94.0 mm to (79.9, 80.0)
- moved R4 91.5 mm to (64.0, 85.2)
- moved D1 90.9 mm to (54.9, 81.0)
- moved R6 90.3 mm to (72.0, 82.1), turned to 90 degrees
- moved C5 89.9 mm to (58.8, 79.0)
- moved C4 89.9 mm to (58.8, 82.9)
- moved D6 79.6 mm to (54.2, 109.6), turned to 90 degrees
- moved Q1 77.3 mm to (74.2, 107.2), turned to 90 degrees
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Connections:
- net /Connector/OBD-CAN_Switch renamed /Connector/~OBD~\CAN
- C2 pad 1: /Connector/OBD_VDD -> Net-(C2-Pad1)
- C3 pad 1: +5V -> Net-(C3-Pad1)
- C5 pad 1: /CAN_Transceiver/BUS_L -> GND
- C5 pad 2: GND -> /CAN_Transceiver/BUS_L
- IC1 pad 8: GND -> Net-(IC1-Pad8)
- J1 pad 1: Net-(J1-Pad1) -> (no net)
- J1 pad 11: Net-(J1-Pad11) -> (no net)
- J1 pad 3: Net-(J1-Pad3) -> (no net)
- J1 pad 5: Net-(J1-Pad5) -> (no net)
- J1 pad 7: Net-(J1-Pad7) -> (no net)
- J1 pad 9: Net-(J1-Pad9) -> (no net)
- J2 pad 10: Net-(J2-Pad10) -> (no net)
- J3 pad 0: (no net) -> GND
- J3 pad 1: Net-(J3-Pad1) -> (no net)
- J3 pad 4: Net-(J3-Pad4) -> (no net)
- J3 pad 6: Net-(J3-Pad6) -> (no net)
- J3 pad 8: Net-(J3-Pad8) -> (no net)
- L1 pad 2: +5V -> Net-(C3-Pad1)
- R1 pad 1: /Connector/OBD_VDD -> Net-(C16-Pad1)
- R3 pad 1: +5V -> Net-(C3-Pad1)
- U1 pad 2: /Connector/OBD_VDD -> Net-(C2-Pad1)
- U1 pad 3: /Connector/OBD_VDD -> Net-(C2-Pad1)
- U1 pad 5: GND -> Net-(R19-Pad2)
- U1 pad 6: +5V -> Net-(C3-Pad1)
- U2 pad 1: Net-(U2-Pad1) -> (no net)
- U2 pad 16: Net-(U2-Pad16) -> (no net)
- U2 pad 17: Net-(U2-Pad17) -> (no net)
- U2 pad 18: Net-(U2-Pad18) -> (no net)
- U2 pad 19: Net-(U2-Pad19) -> (no net)
- U2 pad 2: Net-(U2-Pad2) -> (no net)
- U2 pad 24: Net-(U2-Pad24) -> (no net)
- U2 pad 25: Net-(U2-Pad25) -> (no net)
- U2 pad 3: Net-(U2-Pad3) -> (no net)
- U2 pad 4: Net-(U2-Pad4) -> (no net)
Routing:
- net +3V3: track 111.9 -> 204.1 mm
- net /MCU/Indicator_STA_Mode: track 25.7 -> 96.9 mm
- net /MCU/OBD_Voltage_Check: track 93.0 -> 23.8 mm
- net /MCU/WiFi_Mode: track 57.1 -> 125.4 mm
- net /MCU/Indicator_AP_Mode: track 36.1 -> 103.8 mm
- net +5V: track 52.1 -> 115.0 mm
- net /Connector/OBD_VDD: track 26.5 -> 83.0 mm
- net /CAN_Transceiver/CAN_Tx: track 43.3 -> 8.59 mm
- net /MCU/GPIO_4: track 22.5 -> 49.9 mm
- net /MCU/MTDO: track 73.9 -> 100.2 mm
- net /MCU/GPIO_1: track 36.4 -> 10.3 mm
- net Net-(C12-Pad1): track 100.5 -> 79.9 mm, vias 0 -> 1
- net /MCU/GPIO_3: track 18.8 -> 36.4 mm
- net Net-(C3-Pad1): track 0.00 -> 17.0 mm
- net GND: track 16.4 -> 0.00 mm, vias 14 -> 57
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Other:
- board size 123.2 x 44.5 mm -> 150.1 x 51.8 mm
- board text added: "+12V"
- board text added: "+5V"
- board text added: "ESP-CAN Interface"
- board text added: "Filter"
- board text added: "I/O"
- board text added: "NewTec GmbH. Gabryel Reyes"
- board text added: "~OBD~\CAN Switch"

Commit message: Board Version 6
Parts:
- added C17: 100n, Capacitor_SMD:C_0603_1608Metric_Pad1.05x0.95mm_HandSolder, F.Cu at (79.9, 76.3)
- added L3: 5u, Board:INDPM5550X300N, F.Cu at (129.1, 99.9)
- added REF**: MountingHole_3.2mm_M3_Pad_Via, MountingHole:MountingHole_3.2mm_M3_Pad_Via, F.Cu at (203.3, 61.5)
- added REF**: MountingHole_3.2mm_M3_Pad_Via, MountingHole:MountingHole_3.2mm_M3_Pad_Via, F.Cu at (203.3, 126.5)
- added REF**: MountingHole_3.2mm_M3_Pad_Via, MountingHole:MountingHole_3.2mm_M3_Pad_Via, F.Cu at (43.3, 61.5)
- added REF**: MountingHole_3.2mm_M3_Pad_Via, MountingHole:MountingHole_3.2mm_M3_Pad_Via, F.Cu at (43.3, 126.5)
- L1: footprint Capacitor_SMD:C_0603_1608Metric_Pad1.05x0.95mm_HandSolder -> Board:INDPM5550X300N
- U1: value TPS62170DGK -> TPS62160DGK
- moved L1 4.77 mm to (147.7, 100.1), turned to 0 degrees
- moved FB1 4.00 mm to (135.9, 104.4)
- moved C1 3.76 mm to (134.4, 108.0)
- moved C16 3.76 mm to (132.1, 107.9)
- moved C2 3.76 mm to (136.7, 108.0)
- moved C9 3.76 mm to (134.4, 107.9)
- moved D8 3.76 mm to (128.8, 107.7)
- moved F1 3.76 mm to (122.4, 107.5)
- moved R1 3.76 mm to (131.7, 108.1)
- moved R2 3.76 mm to (137.3, 107.9)
- moved U1 3.59 mm to (145.6, 106.4)
- moved R4 2.11 mm to (64.3, 83.1)
- moved D1 2.06 mm to (56.8, 80.3)
- moved R5 1.55 mm to (64.3, 77.4)
- moved C4 1.19 mm to (59.6, 82.0), turned to 270 degrees
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Routing:
- net +3V3: track 204.1 -> 0.00 mm
- net /MCU/WiFi_Mode: track 125.4 -> 0.00 mm
- net +5V: track 115.0 -> 0.00 mm
- net /MCU/Indicator_AP_Mode: track 103.8 -> 0.00 mm
- net /MCU/MTDO: track 100.2 -> 0.00 mm, vias 1 -> 0
- net /MCU/Indicator_STA_Mode: track 96.9 -> 0.00 mm
- net /MCU/Indicator_Error: track 88.6 -> 0.00 mm
- net /Connector/OBD_VDD: track 83.0 -> 0.00 mm
- net /MCU/MTCK: track 81.5 -> 0.00 mm, vias 1 -> 0
- net Net-(C12-Pad1): track 79.9 -> 0.00 mm, vias 1 -> 0
- net /MCU/MTDI: track 77.1 -> 0.00 mm, vias 1 -> 0
- net /MCU/MTMS: track 67.2 -> 0.00 mm, vias 1 -> 0
- net /MCU/GPIO_4: track 49.9 -> 0.00 mm
- net /Connector/~OBD~\CAN: track 47.2 -> 0.00 mm
- net /MCU/GPIO_3: track 36.4 -> 0.00 mm
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Other:
- board size 150.1 x 51.8 mm -> 170 x 75 mm
- board text removed: "ESP-CAN Interface"
- board text removed: "NewTec GmbH. Gabryel Reyes"

Commit message: Board Version 7
Parts:
- removed REF** (x4): MountingHole_3.2mm_M3_Pad_Via, MountingHole:MountingHole_3.2mm_M3_Pad_Via
- C11, C12, C13, C14, C15, C17, C4, C5, C6, C7, D1, D2, IC1, L2, R10, R11, R12, R21, R4, R5, R6, R7, R9: moved to B.Cu
- J1: value 2606-3356 -> Conn_01x08_Female; footprint Board:2606-3356 -> Board:AST 045-08
- moved R13 95.6 mm to (96.1, 67.6)
- moved R14 91.6 mm to (101.2, 67.6), turned to 90 degrees
- moved D4 89.5 mm to (101.2, 70.9), turned to 270 degrees
- moved C10 86.3 mm to (81.4, 71.8)
- moved FB2 86.3 mm to (80.5, 69.2)
- moved R3 85.4 mm to (75.3, 68.1), turned to 90 degrees
- moved U1 84.6 mm to (70.2, 68.2)
- moved C3 84.0 mm to (79.3, 72.6)
- moved D3 83.4 mm to (96.1, 70.9), turned to 270 degrees
- moved R19 83.3 mm to (76.9, 69.9), turned to 270 degrees
- moved R20 83.3 mm to (76.9, 73.4)
- moved SW1 81.9 mm to (114.6, 68.0), turned to 0 degrees
- moved L1 80.1 mm to (72.2, 73.2)
- moved R15 80.1 mm to (106.2, 67.6), turned to 90 degrees
- moved D5 77.8 mm to (106.2, 70.9), turned to 270 degrees
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Connections:
- J1 pad 1: (no net) -> +3V3
- J1 pad 2: /MCU/GPIO_1 -> GND
- J1 pad 3: (no net) -> /MCU/GPIO_1
- J1 pad 5: (no net) -> /MCU/GPIO_3
- J1 pad 6: /MCU/GPIO_3 -> /MCU/GPIO_4
- J1 pad 8: /MCU/GPIO_4 -> (no net)
- K2 pad 11: /Connector/Pin_3 -> /Connector/Pin_5
- K2 pad 13: /CAN_Transceiver/BUS_H -> /CAN_Transceiver/BUS_L
- K2 pad 4: /CAN_Transceiver/BUS_L -> /CAN_Transceiver/BUS_H
- K2 pad 6: /Connector/Pin_5 -> /Connector/Pin_3
- K2 pad 8: /Connector/Pin_2 -> /Connector/Pin_7
- K2 pad 9: /Connector/Pin_7 -> /Connector/Pin_2
Routing:
- net +5V: track 0.00 -> 143.0 mm, vias 0 -> 1
- net +3V3: track 0.00 -> 112.8 mm
- net Net-(C2-Pad1): track 0.00 -> 58.1 mm
- net /MCU/WiFi_Mode: track 0.00 -> 51.5 mm
- net /Connector/~OBD~\CAN: track 0.00 -> 44.7 mm
- net Net-(D7-Pad2): track 0.00 -> 42.1 mm
- net GND: track 0.00 -> 40.7 mm, vias 38 -> 42
- net /Connector/CAN_Mode: track 0.00 -> 37.7 mm
- net /Connector/Pin_2: track 0.00 -> 29.2 mm
- net /MCU/MTMS: track 0.00 -> 23.7 mm
- net /CAN_Transceiver/CAN_Tx: track 0.00 -> 23.1 mm
- net /Connector/OBD_VDD: track 0.00 -> 22.4 mm
- net /Connector/Pin_3: track 0.00 -> 22.4 mm
- net /MCU/Indicator_STA_Mode: track 0.00 -> 20.9 mm
- net /MCU/GPIO_1: track 0.00 -> 19.5 mm
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Other:
- board size 170 x 75 mm -> 87.5 x 70 mm
- board text added: "ESP32 CAN Analyzer"
- board text added: "Gabryel Reyes"
- board text added: "NewTec Gmbh."
- board text added: "Version 1.0 24.11.2020"
- board text removed: "I/O"
- board text removed: "~OBD~\CAN Switch"
