File: Hardware/010_Implementation/connector.sch (KiCad schematic (older format))
At the start: 12 parts, among them J3 DSUB9, K1 G5V-2-DC5, K2 G5V-2-DC5, Q1 BC817

Commit message: Board Version 1.1 Fixed Relay Supply, standard Pins for CAN Transceiver and added CAN high and Low Labels
Connections:
- net +5V renamed Relay_Supply
Changed lines of the file:
@@
-	1    0    0    -1
-$EndComp
-$Comp
-L power:+5V #PWR024
-U 1 1 5FA1A73B
-P 8530 1420
-F 0 "#PWR024" H 8530 1270 50  0001 C CNN
-F 1 "+5V" H 8545 1593 50  0000 C CNN
-F 2 "" H 8530 1420 50  0001 C CNN
-F 3 "" H 8530 1420 50  0001 C CNN
-	1    8530 1420
 	1    0    0    -1
 $EndComp
@@
 Wire Wire Line
 	8795 1470 9341 1470
+Text HLabel 8530 1420 1    50   Input ~ 0
+Relay_Supply
 $EndSCHEMATC
